File: Hardware/RGBWController.kicad_pcb (KiCad board)
At the start: 2 copper layers, 50 x 30 mm, 18 parts, among them CON1 AVR-ISP-6, IC11 ArduinoProMini, P1 RGBW Strip, P2 CONN_01X02, Q1 IRLML2502, Q2 IRLML2502, Q3 IRLML2502, Q4 IRLML2502, U1 NRF24L01, U2 AMS1117

Commit message: better update with new gerber files
Parts:
- removed IC11: ArduinoProMini, mysensors_arduino:pro_mini
- added IC1: ArduinoProMini, mysensors_arduino:pro_mini, F.Cu at (121.9, 80.0)
- moved Q2 1.27 mm to (124.5, 82.5), turned to 0 degrees
- moved Q1 1.27 mm to (120.7, 82.5), turned to 0 degrees
- moved Q3 1.27 mm to (128.3, 82.5), turned to 0 degrees
- moved Q4 1.27 mm to (132.1, 82.5), turned to 0 degrees
Connections:
- Q1 pad 1: Net-(P1-Pad2) -> R
- Q1 pad 2: R -> GND
- Q1 pad 3: GND -> Net-(P1-Pad2)
- Q2 pad 1: Net-(P1-Pad3) -> G
- Q2 pad 2: G -> GND
- Q2 pad 3: GND -> Net-(P1-Pad3)
- Q3 pad 1: Net-(P1-Pad4) -> B
- Q3 pad 2: B -> GND
- Q3 pad 3: GND -> Net-(P1-Pad4)
- Q4 pad 1: Net-(P1-Pad5) -> W
- Q4 pad 2: W -> GND
- Q4 pad 3: GND -> Net-(P1-Pad5)
Routing:
- net GND: track 110.5 -> 116.2 mm
- net B: track 23.0 -> 28.3 mm
- net W: track 22.1 -> 25.6 mm
- net G: track 23.6 -> 27.2 mm
- net Net-(P1-Pad4): track 11.7 -> 13.2 mm
- net Net-(P1-Pad5): track 13.8 -> 12.5 mm
- net R: track 19.4 -> 20.4 mm
- net Net-(P1-Pad3): track 12.5 -> 13.5 mm
